File: kicad/project/project.kicad_pcb (KiCad board)
At the start: 2 copper layers, 98 x 60 mm, 48 parts, among them J1 SWD, J3 Voltmeter, U1 ADS1015, U2 AP7380, U3 STM32L031F4Px, U4 VN7003ALH

Commit message: Start of layout
Parts:
- removed C11: 10uF, Capacitor_SMD:C_0603_1608Metric_Pad1.05x0.95mm_HandSolder
- removed J3: Voltmeter, theapi:Voltmeter_Header_1x03
- removed R13, R17: 10K, Resistor_SMD:R_0603_1608Metric_Pad1.05x0.95mm_HandSolder
- removed R14: 620K, Resistor_SMD:R_0603_1608Metric_Pad1.05x0.95mm_HandSolder
- removed R15: 100K, Resistor_SMD:R_0603_1608Metric_Pad1.05x0.95mm_HandSolder
- removed R16: SENSE, Resistor_SMD:R_0805_2012Metric_Pad1.15x1.40mm_HandSolder
- removed REF** (x2): TheApiLogo, theapi:TheApiLogoSmall
- removed REF**: TheApiLogoTiny, theapi:TheApiLogoTiny
- removed TP1: TestPoint, TestPoint:TestPoint_Pad_D1.0mm
- removed U3: STM32L031F4Px, Package_SO:TSSOP-20_4.4x6.5mm_P0.65mm
- removed U4: VN7003ALH, theapi:Octapak
- added D6: LED, LED_SMD:LED_0805_2012Metric_Pad1.15x1.40mm_HandSolder, F.Cu at (23.4, 45.6)
- added Q1: MMBT3906, Package_TO_SOT_SMD:SOT-23, F.Cu at (171.0, 56.2)
- added Q2: MMBT3906, Package_TO_SOT_SMD:SOT-23, F.Cu at (170.4, 62.2)
- added Q3: IRF3205, theapi:TO-220F-3_Horizontal_TabUp, B.Cu at (171.2, 52.8)
- added Q4: MMBT3904, Package_TO_SOT_SMD:SOT-23, F.Cu at (166.7, 62.2)
- added R10: 1K, Resistor_SMD:R_0603_1608Metric_Pad1.05x0.95mm_HandSolder, F.Cu at (48.6, 43.6)
- BT1: value Battery_Meter -> Battery; footprint theapi:TerminalBlock_Meter -> TerminalBlock:TerminalBlock_bornier-2_P5.08mm
- C1: value 10uF -> 0.1uF
- C10: value 0.1uF -> 220pF
- C2: value 0.1UF -> 47nF
- C3: value 1uF -> 10uF
- C4: value 10uF -> 47nF
- C6: value 0.1uF -> 10uF; moved to B.Cu
- C7, C9: moved to B.Cu
- C8: value 1uF -> 0.1uF; moved to B.Cu
- D1: value LED -> BAW56; footprint LED_SMD:LED_0805_2012Metric_Pad1.15x1.40mm_HandSolder -> Package_TO_SOT_SMD:SOT-23; moved to F.Cu
- D2: value LED -> BAV99; footprint LED_SMD:LED_0805_2012Metric_Pad1.15x1.40mm_HandSolder -> Package_TO_SOT_SMD:SOT-23; moved to F.Cu
- D3: value LED -> 1N4148; footprint LED_SMD:LED_0805_2012Metric_Pad1.15x1.40mm_HandSolder -> Diode_SMD:D_SOD-123; moved to F.Cu
- D4, J1: moved to F.Cu
- D5: value D_Schottky -> LED; footprint Diode_THT:D_DO-201AD_P12.70mm_Horizontal -> LED_SMD:LED_0805_2012Metric_Pad1.15x1.40mm_HandSolder; moved to F.Cu
- R1, R2: value 220 -> 620K
- R11: value 10K -> 1K; moved to F.Cu
- R12: value 10K -> 220K; moved to F.Cu
- R3, R4: value 10K -> 220K
- R5, R6: value 10K -> 100K
- R7: value 220 -> 4K7
- R8: value 620K -> 10K; moved to B.Cu
- R9: value 100K -> 1K
- U1: value ADS1015 -> NCV4264-2CST33T3G; footprint theapi:TSSOP-10_3x3mm_P0.5mm -> Package_TO_SOT_SMD:SOT-223-3_TabPin2
- U2: value AP7380 -> STM32L031F4Px; footprint Package_TO_SOT_SMD:SOT-23-5_HandSoldering -> Package_SO:TSSOP-20_4.4x6.5mm_P0.65mm
- moved J1 173.8 mm to (23.3, 25.1), turned to 0 degrees
- moved H4 165.0 mm to (43.5, 42.1)
- moved R9 146.4 mm to (59.3, 32.5)
- moved H2 142.3 mm to (47.2, 34.8)
- moved R2 133.5 mm to (52.4, 37.6), turned to 0 degrees
- moved R1 126.2 mm to (59.1, 34.6), turned to 0 degrees
- moved R11 121.8 mm to (55.7, 37.6)
- moved H3 112.7 mm to (49.7, 26.8)
- moved C10 107.8 mm to (55.7, 36.1), turned to 0 degrees
- moved D5 105.7 mm to (27.1, 34.9)
- moved R6 104.5 mm to (52.0, 39.1), turned to 0 degrees
- moved R5 104.2 mm to (55.3, 39.1), turned to 0 degrees
- moved U1 103.3 mm to (123.5, 20.5), turned to 90 degrees
- moved C1 96.7 mm to (121.6, 26.5), turned to 0 degrees
- moved BT1 95.5 mm to (165.5, 46.5), turned to 180 degrees
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Connections:
- BT1 pad 1: /DIODE -> /BATT
- C1 pad 1: +24V -> /REG_IN
- C10 pad 1: +24V -> /BATT_SENSE
- C2 pad 1: +3V3 -> Net-(C2-Pad1)
- C2 pad 2: GND -> pump1
- C3 pad 1: +24V -> +3V3
- C4 pad 1: +3V3 -> Net-(C4-Pad1)
- C4 pad 2: GND -> pump2
- C5 pad 1: +3V3 -> /V_GATE
- C9 pad 1: /BATT_SENSE -> +3V3
- D1 pad 1: GND -> /REG_IN
- D1 pad 2: Net-(D1-Pad2) -> Net-(C2-Pad1)
- D2 pad 1: GND -> Net-(C2-Pad1)
- D2 pad 2: Net-(D2-Pad2) -> /V_GATE
- D3 pad 1: GND -> Net-(D3-Pad1)
- D4 pad 2: /LED_4 -> /LED_1
- D5 pad 1: /DIODE -> GND
- D5 pad 2: /OUT -> /LED_2
- R1 pad 1: Net-(D1-Pad2) -> /SOLAR
- R1 pad 2: /LED_1 -> /PANEL_SENSE
- R11 pad 1: /INPUT -> /LED_2
- R11 pad 2: /PWM -> Net-(R11-Pad2)
- R12 pad 1: /FR_DIAG -> Net-(Q4-Pad2)
- R12 pad 2: Net-(R12-Pad2) -> GND
- R2 pad 1: Net-(D2-Pad2) -> /BATT
- R2 pad 2: /LED_2 -> /BATT_SENSE
- R3 pad 1: Net-(R3-Pad1) -> /V_GATE
- R3 pad 2: GND -> Net-(Q2-Pad1)
- R4 pad 1: +3V3 -> /BATT
- R4 pad 2: SDA -> Net-(D3-Pad2)
- R5 pad 1: +3V3 -> /PANEL_SENSE
- R5 pad 2: SCL -> GND
- R6 pad 1: +3V3 -> /BATT_SENSE
- R6 pad 2: ADC_RDY -> GND
- R7 pad 1: Net-(D3-Pad2) -> Net-(Q3-Pad1)
- R7 pad 2: /LED_3 -> Net-(D3-Pad1)
- R8 pad 1: +24V -> Net-(R8-Pad1)
- R8 pad 2: /PANEL_SENSE -> GND
- R9 pad 1: /PANEL_SENSE -> /LED_1
- R9 pad 2: GND -> Net-(R9-Pad2)
- SC1 pad 1: +24V -> /SOLAR
- U1 pad 1: GND -> /REG_IN
- U1 pad 2: ADC_RDY -> GND
- U1 pad 3: GND -> +3V3
- U2 pad 1: +24V -> Net-(R8-Pad1)
- U2 pad 2: GND -> Net-(R9-Pad2)
- U2 pad 3: +24V -> Net-(R11-Pad2)
- U2 pad 4: Net-(U2-Pad4) -> NRST
Routing:
- net GND: track 182.0 -> 14.9 mm, vias 13 -> 0
- net +24V: track 150.6 -> 0.00 mm, vias 30 -> 0
- net /LED_3: track 122.2 -> 0.00 mm, vias 3 -> 0
- net /BATT_SENSE: track 110.3 -> 0.00 mm, vias 1 -> 0
- net +3V3: track 119.8 -> 14.8 mm
- net /PANEL_SENSE: track 97.1 -> 0.00 mm, vias 1 -> 0
- net ADC_RDY: track 70.7 -> 0.00 mm, vias 3 -> 0
- net SCL: track 63.0 -> 0.00 mm, vias 3 -> 0
- net /OUT: track 62.4 -> 0.00 mm
- net SDA: track 62.3 -> 0.00 mm, vias 5 -> 0
- net CURRENT_SENSE: track 62.3 -> 0.00 mm, vias 3 -> 0
- net /LED_1: track 48.0 -> 0.00 mm, vias 1 -> 0
- net /LED_2: track 44.9 -> 0.00 mm, vias 1 -> 0
- net NRST: track 36.7 -> 0.00 mm, vias 2 -> 0
- net /FR_DIAG: track 36.2 -> 0.00 mm, vias 2 -> 0
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- removed copper zone on B.Cu, net +24V
- removed copper zone on F.Cu, net +24V
- removed copper zone on B.Cu, net -BATT
- removed copper zone on B.Cu, net /DIODE
- removed copper zone on B.Cu, net /OUT
- removed copper zone on B.Cu, net GND
- removed copper zone on F.Cu, net GND
Other:
- board outline removed
- board text added: "TAB UP"
- board text removed: "+ BATTERY -"
- board text removed: "- SOLAR +"
- board text removed: "03/2019 /theapi/pwm-charge-controller v1.0"
- board text removed: "3V3"
- board text removed: "AMMETER"
- board text removed: "BLK"
- board text removed: "CLK"
- board text removed: "DIO"
- board text removed: "GND"
- board text removed: "PWM"
- board text removed: "PWM Charge Controller"
- board text removed: "PWR"
- board text removed: "RED"
- board text removed: "RST"
- board text removed: "TX"
- board text removed: "VOLT METER"

Commit message: Initial board layout
Parts:
- C10, C2, C4, C5, D1, D2, R1, R10, R11, R2, R5, R6, R9: moved to B.Cu
- R7: value 4K7 -> 1K
- moved J1 139.2 mm to (146.1, 90.7)
- moved D6 135.3 mm to (142.8, 109.5), turned to 180 degrees
- moved D5 133.3 mm to (137.5, 109.5), turned to 180 degrees
- moved D4 125.7 mm to (132.0, 109.5), turned to 180 degrees
- moved H1 120.6 mm to (137.5, 116.2)
- moved R10 115.0 mm to (142.9, 109.5), turned to 180 degrees
- moved R11 108.9 mm to (137.5, 109.5)
- moved R9 105.9 mm to (132.0, 109.5)
- moved R6 90.8 mm to (129.2, 86.8)
- moved C10 90.4 mm to (129.2, 88.8)
- moved R2 90.2 mm to (129.2, 84.8), turned to 180 degrees
- moved R1 85.1 mm to (129.2, 82.8), turned to 180 degrees
- moved R5 84.9 mm to (129.2, 80.8)
- moved C5 62.0 mm to (129.3, 91.4)
- moved C4 61.4 mm to (128.5, 94.0), turned to 270 degrees
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Routing:
- net /BATT: track 24.0 -> 13.1 mm, vias 1 -> 0
- net Net-(Q3-Pad1): track 6.38 -> 0.00 mm
- net /V_GATE: track 5.41 -> 1.78 mm
Other:
- board outline added: 23 x 60 mm

Commit message: Connected
Parts:
- removed H2, H3, H4: MountingHole_Pad, MountingHole:MountingHole_3.2mm_M3_Pad
- moved D1 20.2 mm to (127.6, 78.0), turned to 180 degrees
- moved C2 19.8 mm to (130.3, 78.1), turned to 90 degrees
- moved R5 16.5 mm to (129.9, 97.2), turned to 270 degrees
- moved C10 12.7 mm to (128.6, 101.4), turned to 270 degrees
- moved D2 12.7 mm to (127.6, 81.8), turned to 180 degrees
- moved C4 12.3 mm to (130.3, 81.8), turned to 90 degrees
- moved R1 10.7 mm to (129.9, 93.4), turned to 270 degrees
- moved R6 10.7 mm to (127.1, 97.2), turned to 270 degrees
- moved R2 8.94 mm to (127.1, 93.4), turned to 270 degrees
- moved C5 6.89 mm to (129.5, 84.5), turned to 0 degrees
- moved R3 5.87 mm to (139.5, 83.1), turned to 0 degrees
- moved R12 4.91 mm to (143.2, 83.1), turned to 180 degrees
- moved Q2 4.74 mm to (139.5, 85.9), turned to 270 degrees
- moved Q4 3.48 mm to (143.2, 85.9), turned to 90 degrees
- moved H1 0.84 mm to (137.5, 117.1)
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Routing:
- net GND: track 14.9 -> 77.1 mm, vias 0 -> 7
- net /BATT: track 13.1 -> 63.7 mm
- net +3V3: track 14.8 -> 55.7 mm, vias 2 -> 4
- net pump1: track 0.00 -> 38.6 mm, vias 0 -> 3
- net pump2: track 0.00 -> 34.1 mm, vias 0 -> 3
- net /PWM: track 0.00 -> 26.8 mm, vias 0 -> 1
- net Net-(R11-Pad2): track 0.00 -> 24.3 mm, vias 0 -> 1
- net /SOLAR: track 13.6 -> 36.2 mm
- net NRST: track 0.00 -> 22.5 mm, vias 0 -> 1
- net Net-(R9-Pad2): track 0.00 -> 21.9 mm, vias 0 -> 1
- net UART_TX: track 0.00 -> 20.1 mm, vias 0 -> 1
- net /V_GATE: track 1.78 -> 20.2 mm, vias 0 -> 1
- net /REG_IN: track 3.04 -> 17.2 mm, vias 0 -> 1
- net /BATT_SENSE: track 0.00 -> 12.9 mm, vias 0 -> 1
- net /PANEL_SENSE: track 0.00 -> 8.69 mm, vias 0 -> 1
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- added copper zone on B.Cu, net GND
- added copper zone on F.Cu, net GND
